File: nucleo_driver_breakout/untitled.kicad_sch (KiCad schematic)
At the start: 13 parts, among them J5 USB_C_Receptacle_USB2.0_16P, U4 USB3300-EZK, Y1 Crystal

Commit message: changed usb connector and added LCSC IDs
Parts:
- C10, C11: LCSC ID (none) -> C1512022
- C12, C9: LCSC ID (none) -> C1525
- C19: LCSC ID (none) -> C695126
- C7, C8: LCSC ID (none) -> C2858031
- J5: footprint Connector_USB:USB_C_Receptacle_Amphenol_12401610E4-2A -> Connector_USB:USB_C_Receptacle_G-Switch_GT-USB-7010ASV; LCSC ID (none) -> C2988369
- R19: LCSC ID (none) -> C25752
- R39: LCSC ID (none) -> C25744
- U4: LCSC ID (none) -> C108383
- Y1: LCSC ID (none) -> C1985382
Changed lines of the file:
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@@
+			)
+		)
+		(property "LCSC ID" "C1525"
+			(at 167.64 59.69 0)
+			(effects
+				(font
+					(size 1.27 1.27)
+				)
+				(hide yes)
 			)
 		)
@@
 			)
 		)
+		(property "LCSC ID" "C2858031"
+			(at 187.96 67.31 0)
+			(effects
+				(font
+					(size 1.27 1.27)
+				)
+				(hide yes)
+			)
+		)
 		(pin "2"
 		)
@@
 			)
 		)
+		(property "LCSC ID" "C108383"
+			(at 160.02 93.98 0)
+			(effects
+				(font
+					(size 1.27 1.27)
+				)
+				(hide yes)
+			)
+		)
 		(pin "3"
 		)
@@
 			)
 		)
+		(property "LCSC ID" "C1525"
+			(at 72.39 104.14 0)
+			(effects
+				(font
+					(size 1.27 1.27)
+				)
+				(hide yes)
+			)
+		)
 		(pin "2"
 		)
@@
 			)
 		)
-		(property "Footprint" "Connector_USB:USB_C_Receptacle_Amphenol_12401610E4-2A"
+		(property "Footprint" "Connector_USB:USB_C_Receptacle_G-Switch_GT-USB-7010ASV"
 			(at 83.82 74.93 0)
 			(effects
@@
 			)
 		)
-		(property "Datasheet" "https://www.usb.org/sites/default/files/documents/usb_type-c.zip"
+		(property "Datasheet" "https://www.lcsc.com/product-detail/USB-Connectors_G-Switch-GT-USB-7010ASV_C2988369.html"
 			(at 83.82 74.93 0)
 			(effects
@@
 			)
 		)
-		(property "Description" "USB 2.0-only 16P Type-C Receptacle connector"
+		(property "Description" "USB 2.0 3A 1 260℃ Surface Mount，Right Angle 16P Female -40℃~+85℃ Gold High Conductivity Copper Type-C SMD USB Connectors ROHS "
+			(at 80.01 74.93 0)
+			(effects
+				(font
+					(size 1.27 1.27)
+				)
+				(hide yes)
+			)
+		)
+		(property "LCSC ID" "C2988369"
 			(at 80.01 74.93 0)
 			(effects
@@
 		)
 		(property "Description" "Unpolarized capacitor"
+			(at 100.33 48.26 0)
+			(effects
+				(font
+					(size 1.27 1.27)
+				)
+				(hide yes)
+			)
+		)
+		(property "LCSC ID" "C695126"
 			(at 100.33 48.26 0)
 			(effects
@@
 			)
 		)
+		(property "LCSC ID" "C1512022"
+			(at 115.57 101.6 0)
+			(effects
+				(font
+					(size 1.27 1.27)
+				)
+				(hide yes)
+			)
+		)
 		(pin "2"
 		)
@@
 			)
 		)
+		(property "LCSC ID" "C1512022"
+			(at 109.22 91.44 0)
+			(effects
+				(font
+					(size 1.27 1.27)
+				)
+				(hide yes)
+			)
+		)
 		(pin "2"
 		)
@@
 			)
 		)
+		(property "LCSC ID" "C1985382"
+			(at 124.46 91.44 0)
+			(effects
+				(font
+					(size 1.27 1.27)
+				)
+				(hide yes)
+			)
+		)
 		(pin "1"
 		)
@@
 			)
 		)
+		(property "LCSC ID" "C2858031"
+			(at 203.2 67.31 0)
+			(effects
+				(font
+					(size 1.27 1.27)
+				)
+				(hide yes)
+			)
+		)
 		(pin "2"
 		)
@@
 			)
 		)
+		(property "LCSC ID" "C25744"
+			(at 124.46 66.04 0)
+			(effects
+				(font
+					(size 1.27 1.27)
+				)
+				(hide yes)
+			)
+		)
 		(pin "2"
 		)
@@
 			(at 127 119.38 0)
 			(effects
+				(font
+					(size 1.27 1.27)
+				)
+				(hide yes)
+			)
+		)
+		(property "LCSC ID" "C25752"
+			(at 127 119.38 0)
+			(effects

Commit message: added bolt holes, vias, and fixed some silkscreen overlaps
Parts:
- C19: value 3.3u -> 4.7u
Changed lines of the file:
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@@
 			)
 		)
-		(property "Value" "3.3u"
+		(property "Value" "4.7u"
 			(at 93.98 49.022 0)
 			(effects
